File: Production Files/FTDI_SmartBasic-GiantPanel-v10a.brd (EAGLE design)
At the start: 341.9 x 235.2 mm, 2252 parts, among them U1 FT232RLSSOP, U10 TS3USB221A, U100 TS3USB221A, U101 FT232RLSSOP, U102 MIC5219 3.3V, U103 TS3USB221A, U104 FT232RLSSOP, U105 MIC5219 3.3V, U106 TS3USB221A, U107 FT232RLSSOP, U108 MIC5219 3.3V, U109 TS3USB221A, U11 FT232RLSSOP, U110 FT232RLSSOP, U111 MIC5219 3.3V, U112 TS3USB221A, U113 FT232RLSSOP, U114 MIC5219 3.3V, U115 TS3USB221A, U116 FT232RLSSOP, U117 MIC5219 3.3V, U118 TS3USB221A, U119 FT232RLSSOP, U12 MIC5219 3.3V, U120 MIC5219 3.3V, U121 TS3USB221A, U122 FT232RLSSOP, U123 MIC5219 3.3V, U124 TS3USB221A, U125 FT232RLSSOP, U126 MIC5219 3.3V, U127 TS3USB221A, U128 FT232RLSSOP, U129 MIC5219 3.3V, U13 TS3USB221A, U130 TS3USB221A, U131 FT232RLSSOP, U132 MIC5219 3.3V, U133 TS3USB221A, U134 FT232RLSSOP, U135 MIC5219 3.3V, U136 TS3USB221A, U137 FT232RLSSOP, U138 MIC5219 3.3V, U139 TS3USB221A, U14 FT232RLSSOP, U140 FT232RLSSOP, U141 MIC5219 3.3V, U142 TS3USB221A, U143 FT232RLSSOP, U144 MIC5219 3.3V, U145 TS3USB221A, U146 FT232RLSSOP, U147 MIC5219 3.3V, U148 TS3USB221A, U149 FT232RLSSOP, U15 MIC5219 3.3V, U150 MIC5219 3.3V, U151 TS3USB221A, U152 FT232RLSSOP, U153 MIC5219 3.3V, U154 TS3USB221A, U155 FT232RLSSOP, U156 MIC5219 3.3V, U157 TS3USB221A, U158 FT232RLSSOP, U159 MIC5219 3.3V, U16 TS3USB221A, U160 TS3USB221A, U161 FT232RLSSOP, U162 MIC5219 3.3V, U163 TS3USB221A, U164 FT232RLSSOP, U165 MIC5219 3.3V, U166 TS3USB221A, U167 FT232RLSSOP, U168 MIC5219 3.3V, U169 TS3USB221A, U17 FT232RLSSOP, U170 FT232RLSSOP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

Commit message: re-created panel with correct silk
Parts:
- moved E$6 117.9 mm to (166.2, 127.3)
- moved E$7 117.9 mm to (166.2, 108.0)
- moved E$10 98.6 mm to (337.4, 127.3), turned to 0 degrees
- moved E$11 98.6 mm to (337.4, 225.8), turned to 180 degrees
- moved E$2 98.6 mm to (337.4, 9.40), turned to 0 degrees
- moved E$3 98.6 mm to (337.4, 108.0), turned to 180 degrees
- moved E$5 98.6 mm to (166.2, 9.40), turned to 0 degrees
- moved E$8 98.6 mm to (166.2, 225.8), turned to 180 degrees
Other:
- outline, holes or cut-outs redrawn
- board text added: "v11"
- board text removed: "v10"
